File: Hackpad/Hackpad.kicad_sch (KiCad schematic)
At the start: 4 parts, among them SW1 SW_Push, SW2 SW_Push, SW3 SW_Push, U1 MOUDLE-SEEEDUINO-XIAO

Commit message: Iteration #2!
Parts:
- added SW4, SW5, SW6, SW7, SW8, SW9: SW_Push, Button_Switch_Keyboard:SW_Cherry_MX_1.00u_PCB, symbol Switch:SW_Push
Connections:
- net GND: now also SW4.2, SW5.2, SW6.1, SW7.1, SW8.1, SW9.1
- net at U1.1 (PA02_A0_D0): now also SW5.1
- net at U1.2 (PA4_A1_D1): now also SW4.1
- net at U1.3 (PA10_A2_D2): now also SW6.2
- net at U1.4 (PA11_A3_D3): now also SW7.2
- net at U1.5 (PA8_A4_D4_SDA): now also SW8.2
- net at U1.6 (PA9_A5_D5_SCL): now also SW9.2
